File: kicad/LedArray.kicad_pcb (KiCad board)
At the start: 2 copper layers, 83.8 x 29.8 mm, 147 parts, among them J1 HT16K33

Commit message: patched
Parts:
- removed REF** (x2): MountingHole_2.2mm_M2_Pad_Via, MountingHole:MountingHole_2.2mm_M2_Pad_Via
- R6: value 2.2k -> 1.0k
- turned D2 to 0 degrees
- turned D3 to 0 degrees
- turned R6 to 180 degrees
- renumbered USB to USB1
Connections:
- D2 pad 1: /D+ -> Net-(D2-Pad1)
- D3 pad 1: /D- -> Net-(D3-Pad1)
- R4 pad 1: Net-(R4-Pad1) -> Net-(D3-Pad1)
- R5 pad 2: Net-(R5-Pad2) -> Net-(D2-Pad1)
- R6 pad 2: /D- -> Net-(D3-Pad1)
- USB1 pad 2: Net-(R4-Pad1) -> Net-(D3-Pad1)
- USB1 pad 3: Net-(R5-Pad2) -> Net-(D2-Pad1)
Routing:
- net Net-(D3-Pad1): track 0.00 -> 17.4 mm
- net GND: track 45.1 -> 54.4 mm, vias 10 -> 11
- net Net-(D2-Pad1): track 0.00 -> 6.81 mm
- net /D-: track 28.6 -> 22.8 mm
- net Net-(R5-Pad2): track 4.04 -> 0.00 mm
- net Net-(R4-Pad1): track 3.53 -> 0.00 mm
- net /D+: track 20.8 -> 18.5 mm
