File: kicad/LedArray.sch (KiCad schematic (older format))
At the start: 145 parts, among them J1 HT16K33

Commit message: patched
Parts:
- J1: symbol Eurocad:HT16K33 -> LedArray-rescue:HT16K33-Eurocad
- R6: value 2.2k -> 1.0k
Connections:
- net D+: no longer D2.1 (K)
- net D-: no longer D3.1 (K), R6.2
- net at R4.1, USB1.2 (D-): now also D3.1 (K), R6.2
- net at R5.2, USB1.3 (D+): now also D2.1 (K)
Other:
- moved on the sheet: D2, D3, R4, R5, R6
Changed lines of the file:
@@
 L Device:R R4
 U 1 1 6349CD2E
-P 3600 1900
-F 0 "R4" V 3393 1900 50  0000 C CNN
-F 1 "68R" V 3484 1900 50  0000 C CNN
-F 2 "Resistor_SMD:R_0805_2012Metric_Pad1.15x1.40mm_HandSolder" V 3530 1900 50  0001 C CNN
-F 3 "~" H 3600 1900 50  0001 C CNN
-	1    3600 1900
+P 3200 1900
+F 0 "R4" V 2993 1900 50  0000 C CNN
+F 1 "68R" V 3084 1900 50  0000 C CNN
+F 2 "Resistor_SMD:R_0805_2012Metric_Pad1.15x1.40mm_HandSolder" V 3130 1900 50  0001 C CNN
+F 3 "~" H 3200 1900 50  0001 C CNN
+	1    3200 1900
 	0    1    1    0
 $EndComp
@@
 L Device:R R5
 U 1 1 6349DEB4
-P 3600 2000
-F 0 "R5" V 3807 2000 50  0000 C CNN
-F 1 "68R" V 3716 2000 50  0000 C CNN
-F 2 "Resistor_SMD:R_0805_2012Metric_Pad1.15x1.40mm_HandSolder" V 3530 2000 50  0001 C CNN
-F 3 "~" H 3600 2000 50  0001 C CNN
-	1    3600 2000
+P 3200 2000
+F 0 "R5" V 3407 2000 50  0000 C CNN
+F 1 "68R" V 3316 2000 50  0000 C CNN
+F 2 "Resistor_SMD:R_0805_2012Metric_Pad1.15x1.40mm_HandSolder" V 3130 2000 50  0001 C CNN
+F 3 "~" H 3200 2000 50  0001 C CNN
+	1    3200 2000
 	0    -1   -1   0
 $EndComp
-Wire Wire Line
-	3750 1900 4000 1900
-Wire Wire Line
-	3750 2000 4000 2000
 Wire Wire Line
 	4300 1600 4300 1500
@@
 Wire Wire Line
 	4300 1500 4300 1350
-Wire Wire Line
-	2550 1900 3250 1900
-Wire Wire Line
-	3450 2000 3000 2000
 $Comp
 L Device:D_Zener D3
 U 1 1 63869311
-P 3250 2200
-F 0 "D3" V 3204 2279 50  0000 L CNN
-F 1 "3.3V" V 3295 2279 50  0000 L CNN
-F 2 "Diode_SMD:D_SOD-523" H 3250 2200 50  0001 C CNN
-F 3 "~" H 3250 2200 50  0001 C CNN
-	1    3250 2200
+P 3700 2400
+F 0 "D3" V 3654 2479 50  0000 L CNN
+F 1 "3.3V" V 3745 2479 50  0000 L CNN
+F 2 "Diode_SMD:D_SOD-523" H 3700 2400 50  0001 C CNN
+F 3 "~" H 3700 2400 50  0001 C CNN
+	1    3700 2400
 	0    1    1    0
 $EndComp
@@
 L Device:D_Zener D2
 U 1 1 6386A711
-P 3000 2300
-F 0 "D2" V 2954 2379 50  0000 L CNN
-F 1 "3.3V" V 3045 2379 50  0000 L CNN
-F 2 "Diode_SMD:D_SOD-523" H 3000 2300 50  0001 C CNN
-F 3 "~" H 3000 2300 50  0001 C CNN
-	1    3000 2300
+P 3450 2500
+F 0 "D2" V 3404 2579 50  0000 L CNN
+F 1 "3.3V" V 3495 2579 50  0000 L CNN
+F 2 "Diode_SMD:D_SOD-523" H 3450 2500 50  0001 C CNN
+F 3 "~" H 3450 2500 50  0001 C CNN
+	1    3450 2500
 	0    1    1    0
 $EndComp
 Wire Wire Line
-	3000 2150 3000 2000
-Connection ~ 3000 2000
-Wire Wire Line
-	3000 2000 2550 2000
-Wire Wire Line
-	3250 2050 3250 1900
-Connection ~ 3250 1900
-Wire Wire Line
-	3250 1900 3450 1900
-Wire Wire Line
-	3250 2350 3250 2500
-Wire Wire Line
-	3250 2500 3150 2500
-Wire Wire Line
-	3000 2500 3000 2450
-Wire Wire Line
-	3150 2500 3150 2600
-Connection ~ 3150 2500
-Wire Wire Line
-	3150 2500 3000 2500
+	3700 2550 3700 2700
+Wire Wire Line
+	3700 2700 3600 2700
+Wire Wire Line
+	3450 2700 3450 2650
+Wire Wire Line
+	3600 2700 3600 2800
+Connection ~ 3600 2700
+Wire Wire Line
+	3600 2700 3450 2700
 $Comp
 L power:GND #PWR013
 U 1 1 63992610
-P 3150 2600
-F 0 "#PWR013" H 3150 2350 50  0001 C CNN
-F 1 "GND" H 3155 2427 50  0000 C CNN
-F 2 "" H 3150 2600 50  0001 C CNN
-F 3 "" H 3150 2600 50  0001 C CNN
-	1    3150 2600
+P 3600 2800
+F 0 "#PWR013" H 3600 2550 50  0001 C CNN
+F 1 "GND" H 3605 2627 50  0000 C CNN
+F 2 "" H 3600 2800 50  0001 C CNN
+F 3 "" H 3600 2800 50  0001 C CNN
+	1    3600 2800
 	1    0    0    -1
 $EndComp
@@
 L Device:R R6
 U 1 1 6402D61C
-P 3250 1700
-F 0 "R6" H 3320 1746 50  0000 L CNN
-F 1 "2.2k" H 3320 1655 50  0000 L CNN
-F 2 "Resistor_SMD:R_0805_2012Metric_Pad1.15x1.40mm_HandSolder" V 3180 1700 50  0001 C CNN
-F 3 "~" H 3250 1700 50  0001 C CNN
-	1    3250 1700
-	1    0    0    -1
-$EndComp
-Wire Wire Line
-	3250 1850 3250 1900
+P 3600 1700
+F 0 "R6" H 3670 1746 50  0000 L CNN
+F 1 "1.0k" H 3670 1655 50  0000 L CNN
+F 2 "Resistor_SMD:R_0805_2012Metric_Pad1.15x1.40mm_HandSolder" V 3530 1700 50  0001 C CNN
+F 3 "~" H 3600 1700 50  0001 C CNN
+	1    3600 1700
+	1    0    0    -1
+$EndComp
+Wire Wire Line
+	3600 1850 3600 1900
 $Comp
 L power:VDD #PWR0102
 U 1 1 6407EFBA
-P 3250 1550
-F 0 "#PWR0102" H 3250 1400 50  0001 C CNN
-F 1 "VDD" H 3267 1723 50  0000 C CNN
-F 2 "" H 3250 1550 50  0001 C CNN
-F 3 "" H 3250 1550 50  0001 C CNN
-	1    3250 1550
+P 3600 1550
+F 0 "#PWR0102" H 3600 1400 50  0001 C CNN
+F 1 "VDD" H 3617 1723 50  0000 C CNN
+F 2 "" H 3600 1550 50  0001 C CNN
+F 3 "" H 3600 1550 50  0001 C CNN
+	1    3600 1550
 	1    0    0    -1
 $EndComp
@@
 	4400 5250 5800 5250
 $Comp
-L Eurocad:HT16K33 J1
+L LedArray-rescue:HT16K33-Eurocad J1
 U 1 1 60C7CDAD
 P 3750 4600
@@
 	3600 1250 3600 1200
 Connection ~ 3800 1250
+Connection ~ 3600 1900
+Wire Wire Line
+	2550 1900 3050 1900
+Wire Wire Line
+	2550 2000 3050 2000
+Wire Wire Line
+	3350 1900 3600 1900
+Wire Wire Line
+	3350 2000 3450 2000
+Wire Wire Line
+	3450 2000 3450 2350
+Connection ~ 3450 2000
+Wire Wire Line
+	3450 2000 4000 2000
+Wire Wire Line
+	3700 2250 3700 1900
+Wire Wire Line
+	3600 1900 3700 1900
+Connection ~ 3700 1900
+Wire Wire Line
+	3700 1900 4000 1900
 $EndSCHEMATC
